File: electronics/Incubator_board/INCUBATOR.brd (EAGLE design)
At the start: 43.7 x 49.2 mm, 10 parts, among them Q1 RFP30N06LE, X1 22-23-2031, X2 22-23-2031

Commit message: changes in the board
Parts:
- removed RESITANCEWIRE1: 22-23-2021, con-molex:22-23-2021
- added 12V_POWER_IN: 22-23-2021, con-molex:22-23-2021
- Q1: device SparkFun:TO220V -> IRF3205:TO254P1041X444X2933-3
- R36: value 100 -> 220
- moved RESITANCEWIRE 29.5 mm to (39.9, 34.6), turned to 90 degrees
- moved Q1 14.9 mm to (33.5, 33.6), turned to 90 degrees
- moved R36 6.71 mm to (31.7, 27.8), turned to 90 degrees
- moved R6 4.47 mm to (33.7, 27.9)
Connections:
- net 12V: now also 12V_POWER_IN.2; no longer RESITANCEWIRE1.2
- net GND: now also 12V_POWER_IN.1; no longer RESITANCEWIRE1.1
Routing:
- net HOTEND-GND: track 58.5 -> 8.98 mm
- net GND: track 0.00 -> 33.7 mm
- net N$71: track 31.6 -> 5.59 mm
- net GPIO16/HEATER: track 13.1 -> 5.57 mm
- net 12V: track 5.56 -> 3.09 mm
- net BME_SCL_SCK/GPIO34: track 10.3 -> 12.2 mm
- net VENT_SERVO/GPIO37: track 15.3 -> 13.5 mm
- net TRAY_SERVO/GPIO38: track 10.6 -> 12.1 mm

Commit message: board updates
Parts:
- Q1: device IRF3205:TO254P1041X444X2933-3 -> TO92127P520H700-3:TO92127P520H700-3
- moved Q1 0.51 mm to (33.6, 33.0)
Connections:
- net GND: now also Q1.S; no longer Q1.3
- net HOTEND-GND: now also Q1.D; no longer Q1.2
- net N$71: now also Q1.G; no longer Q1.1
Routing:
- net GND: track 33.7 -> 40.5 mm
- net N$71: track 5.59 -> 7.10 mm
- net HOTEND-GND: track 8.98 -> 10.5 mm
Changed lines of the file:
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@@
 <attribute name="VALUE" x="3.905" y="45.1" size="0.4064" layer="27" ratio="10" rot="R270"/>
 </element>
-<element name="Q1" library="IRF3205" package="TO254P1041X444X2933-3" value="RFP30N06LE" x="33.51" y="33.56" smashed="yes" rot="R90">
-<attribute name="AVAILABILITY" value="Not in stock" x="33.51" y="33.56" size="1.778" layer="27" rot="R90" display="off"/>
-<attribute name="DESCRIPTION" value=" N-Channel 55V 110A (Tc) 200W (Tc) Through Hole TO-220AB " x="33.51" y="33.56" size="1.778" layer="27" rot="R90" display="off"/>
-<attribute name="MF" value="Infineon Technologies" x="33.51" y="33.56" size="1.778" layer="27" rot="R90" display="off"/>
-<attribute name="MP" value="IRF3205" x="33.51" y="33.56" size="1.778" layer="27" rot="R90" display="off"/>
-<attribute name="NAME" x="30.081" y="30.766" size="1.27" layer="25" ratio="10" rot="R90"/>
-<attribute name="PACKAGE" value="TO-220 Infineon" x="33.51" y="33.56" size="1.778" layer="27" rot="R90" display="off"/>
-<attribute name="PRICE" value="None" x="33.51" y="33.56" size="1.778" layer="27" rot="R90" display="off"/>
+<element name="Q1" library="TO92127P520H700-3" package="TO92127P520H700-3" value="RFP30N06LE" x="33.576578125" y="33.04959375" smashed="yes" rot="R90">
+<attribute name="NAME" x="30.147578125" y="30.25559375" size="1.27" layer="25" ratio="10" rot="R90"/>
 </element>
 <element name="R36" library="ipc-7351-resistor" package="RESC2012X70N" value="220" x="31.67" y="27.78" smashed="yes" rot="R90">
@@
 <signals>
 <signal name="GND" class="1">
-<contactref element="Q1" pad="3"/>
+<contactref element="Q1" pad="S"/>
 <contactref element="R6" pad="2"/>
 <contactref element="JP2" pad="2"/>
@@
 <wire x1="9.87649375" y1="14.617428125" x2="5.84201875" y2="14.617428125" width="0.4572" layer="1"/>
 <wire x1="5.84201875" y1="14.617428125" x2="5.821515625" y2="14.596925" width="0.4572" layer="1"/>
+<wire x1="33.576578125" y1="31.77959375" x2="36.820721875" y2="31.77959375" width="0.4572" layer="1"/>
+<wire x1="36.820721875" y1="31.77959375" x2="36.95260625" y2="31.647709375" width="0.4572" layer="1"/>
+<wire x1="36.95260625" y1="31.647709375" x2="33.7084625" y2="31.647709375" width="0.4572" layer="1"/>
+<wire x1="33.7084625" y1="31.647709375" x2="33.576578125" y2="31.77959375" width="0.4572" layer="1"/>
 </signal>
 <signal name="12V">
@@
 </signal>
 <signal name="HOTEND-GND" class="1">
-<contactref element="Q1" pad="2"/>
+<contactref element="Q1" pad="D"/>
 <contactref element="RESITANCEWIRE" pad="2"/>
 <wire x1="39.7764" y1="37.4904" x2="39.7764" y2="35.8902" width="0.4572" layer="1"/>
 <wire x1="39.3192" y1="37.9476" x2="39.7764" y2="37.4904" width="0.4572" layer="1"/>
-<wire x1="36.1188" y1="37.9476" x2="39.3192" y2="37.9476" width="0.4572" layer="1"/>
-<wire x1="34.7472" y1="36.576" x2="36.1188" y2="37.9476" width="0.4572" layer="1"/>
-<wire x1="34.5186" y1="36.576" x2="34.7472" y2="36.576" width="0.4572" layer="1"/>
-<wire x1="34.0614" y1="36.1188" x2="34.5186" y2="36.576" width="0.4572" layer="1"/>
-<wire x1="33.6042" y1="36.1188" x2="34.0614" y2="36.1188" width="0.4572" layer="1"/>
+<wire x1="36.007834375" y1="37.9476" x2="39.3192" y2="37.9476" width="0.4572" layer="1"/>
+<wire x1="34.547465625" y1="36.48723125" x2="36.007834375" y2="37.9476" width="0.4572" layer="1"/>
+<wire x1="34.42983125" y1="36.48723125" x2="34.547465625" y2="36.48723125" width="0.4572" layer="1"/>
+<wire x1="33.874359375" y1="35.931759375" x2="34.42983125" y2="36.48723125" width="0.4572" layer="1"/>
 <wire x1="39.7764" y1="35.8902" x2="39.94" y2="35.89" width="0.4572" layer="1"/>
-<wire x1="33.6042" y1="36.1188" x2="33.51" y2="36.1" width="0.4572" layer="1"/>
+<wire x1="34.101578125" y1="35.2520125" x2="33.576578125" y2="34.31959375" width="0.4572" layer="1"/>
+<wire x1="34.101578125" y1="35.2520125" x2="33.874359375" y2="35.931759375" width="0.4572" layer="1"/>
 </signal>
 <signal name="N$71">
-<contactref element="Q1" pad="1"/>
+<contactref element="Q1" pad="G"/>
 <contactref element="R36" pad="2"/>
-<wire x1="31.7754" y1="30.4038" x2="31.7754" y2="28.8036" width="0.4572" layer="1"/>
-<wire x1="33.3756" y1="32.004" x2="31.7754" y2="30.4038" width="0.4572" layer="1"/>
-<wire x1="33.3756" y1="33.3756" x2="33.3756" y2="32.004" width="0.4572" layer="1"/>
+<wire x1="31.7754" y1="32.889321875" x2="31.7754" y2="28.8036" width="0.4572" layer="1"/>
+<wire x1="31.9228375" y1="33.036759375" x2="31.7754" y2="32.889321875" width="0.4572" layer="1"/>
 <wire x1="31.7754" y1="28.8036" x2="31.67" y2="28.73" width="0.4572" layer="1"/>
-<wire x1="33.3756" y1="33.3756" x2="33.51" y2="33.56" width="0.4572" layer="1"/>
+<wire x1="33.576578125" y1="33.04959375" x2="34.08874375" y2="33.036759375" width="0.4572" layer="1"/>
+<wire x1="34.08874375" y1="33.036759375" x2="31.9228375" y2="33.036759375" width="0.4572" layer="1"/>
 </signal>
 <signal name="BME_SCL_SCK/GPIO34">
