File: electronics/Incubator_board/INCUBATOR.sch (EAGLE design)
At the start: 10 parts, among them Q1 RFP30N06LE, X1 22-23-2031, X2 22-23-2031

Commit message: changes in the board
Parts:
- Q1: device SparkFun:MOSFET-NCHANNELPTH2 -> IRF3205:IRF3205
- R36: value 100 -> 220
- renumbered RESITANCEWIRE1 to 12V_POWER_IN
Changed lines of the file:
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@@
 <part name="GND20" library="SparkFun" deviceset="GND" device=""/>
 <part name="U$13" library="12v" deviceset="12V" device=""/>
-<part name="Q1" library="SparkFun" deviceset="MOSFET-NCHANNEL" device="PTH2" value="RFP30N06LE"/>
+<part name="Q1" library="IRF3205" deviceset="IRF3205" device="" value="RFP30N06LE"/>
 <part name="R6" library="ipc-7351-resistor" deviceset="RESISTOR_" device="0805" value="100k"/>
 <part name="GND28" library="SparkFun" deviceset="GND" device=""/>
-<part name="R36" library="ipc-7351-resistor" deviceset="RESISTOR_" device="0805" value="100"/>
+<part name="R36" library="ipc-7351-resistor" deviceset="RESISTOR_" device="0805" value="220"/>
 <part name="JP1" library="pinhead" library_urn="urn:adsk.eagle:library:325" deviceset="PINHD-1X7" device="" package3d_urn="urn:adsk.eagle:package:22477/2"/>
 <part name="JP2" library="pinhead" library_urn="urn:adsk.eagle:library:325" deviceset="PINHD-1X7" device="" package3d_urn="urn:adsk.eagle:package:22477/2"/>
@@
 <part name="X1" library="con-molex" library_urn="urn:adsk.eagle:library:165" deviceset="22-23-2031" device="" package3d_urn="urn:adsk.eagle:package:8078634/1"/>
 <part name="X2" library="con-molex" library_urn="urn:adsk.eagle:library:165" deviceset="22-23-2031" device="" package3d_urn="urn:adsk.eagle:package:8078634/1"/>
-<part name="RESITANCEWIRE1" library="con-molex" library_urn="urn:adsk.eagle:library:165" deviceset="22-23-2021" device="" package3d_urn="urn:adsk.eagle:package:8078633/1"/>
+<part name="12V_POWER_IN" library="con-molex" library_urn="urn:adsk.eagle:library:165" deviceset="22-23-2021" device="" package3d_urn="urn:adsk.eagle:package:8078633/1"/>
 </parts>
 <sheets>
@@
 <attribute name="VALUE" x="57.404" y="79.756" size="1.778" layer="96"/>
 </instance>
-<instance part="Q1" gate="G$1" x="50.8" y="68.58" smashed="yes">
-<attribute name="NAME" x="45.72" y="72.39" size="1.778" layer="95"/>
+<instance part="Q1" gate="G$1" x="48.26" y="68.58" smashed="yes">
+<attribute name="NAME" x="43.18" y="72.39" size="1.778" layer="95"/>
 </instance>
 <instance part="R6" gate="G$1" x="33.02" y="60.96" smashed="yes" rot="R270">
@@
 <attribute name="NAME" x="-43.18" y="6.858" size="1.524" layer="95"/>
 </instance>
-<instance part="RESITANCEWIRE1" gate="-1" x="73.66" y="50.8" smashed="yes">
+<instance part="12V_POWER_IN" gate="-1" x="73.66" y="50.8" smashed="yes">
 <attribute name="NAME" x="76.2" y="50.038" size="1.524" layer="95"/>
 <attribute name="VALUE" x="72.898" y="52.197" size="1.778" layer="96"/>
 </instance>
-<instance part="RESITANCEWIRE1" gate="-2" x="73.66" y="48.26" smashed="yes">
+<instance part="12V_POWER_IN" gate="-2" x="73.66" y="48.26" smashed="yes">
 <attribute name="NAME" x="76.2" y="47.498" size="1.524" layer="95"/>
 </instance>
@@
 </segment>
 <segment>
-<pinref part="RESITANCEWIRE1" gate="-1" pin="S"/>
+<pinref part="12V_POWER_IN" gate="-1" pin="S"/>
 <wire x1="71.12" y1="50.8" x2="66.04" y2="50.8" width="0.1524" layer="91"/>
 <label x="66.04" y="50.8" size="1.778" layer="95"/>
@@
 </segment>
 <segment>
-<pinref part="RESITANCEWIRE1" gate="-2" pin="S"/>
+<pinref part="12V_POWER_IN" gate="-2" pin="S"/>
 <wire x1="71.12" y1="48.26" x2="66.04" y2="48.26" width="0.1524" layer="91"/>
 <label x="66.04" y="48.26" size="1.778" layer="95"/>
@@
 <pinref part="Q1" gate="G$1" pin="G"/>
 <pinref part="R36" gate="G$1" pin="2"/>
+<wire x1="43.18" y1="68.58" x2="45.72" y2="66.04" width="0.1524" layer="91"/>
 </segment>
 </net>

Commit message: board updates
Parts:
- Q1: device IRF3205:IRF3205 -> TO92127P520H700-3:TN0702N3-G
Connections:
- net GND: now also Q1.SOURCE; no longer Q1.S
- net HOTEND-GND: now also Q1.DRAIN; no longer Q1.D
- net N$71: now also Q1.GATE; no longer Q1.G
Changed lines of the file:
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@@
 <part name="GND20" library="SparkFun" deviceset="GND" device=""/>
 <part name="U$13" library="12v" deviceset="12V" device=""/>
-<part name="Q1" library="IRF3205" deviceset="IRF3205" device="" value="RFP30N06LE"/>
+<part name="Q1" library="TO92127P520H700-3" deviceset="TN0702N3-G" device="" value="RFP30N06LE"/>
 <part name="R6" library="ipc-7351-resistor" deviceset="RESISTOR_" device="0805" value="100k"/>
 <part name="GND28" library="SparkFun" deviceset="GND" device=""/>
@@
 <wire x1="50.8" y1="63.5" x2="50.8" y2="55.88" width="0.1524" layer="91"/>
 <pinref part="GND20" gate="1" pin="GND"/>
-<pinref part="Q1" gate="G$1" pin="S"/>
+<pinref part="Q1" gate="G$1" pin="SOURCE"/>
 </segment>
 <segment>
@@
 <wire x1="54.61" y1="73.66" x2="54.61" y2="68.58" width="0.1524" layer="91"/>
 <wire x1="54.61" y1="68.58" x2="60.96" y2="68.58" width="0.1524" layer="91"/>
-<pinref part="Q1" gate="G$1" pin="D"/>
+<pinref part="Q1" gate="G$1" pin="DRAIN"/>
 <pinref part="RESITANCEWIRE" gate="-2" pin="S"/>
 </segment>
@@
 <net name="N$71" class="0">
 <segment>
-<pinref part="Q1" gate="G$1" pin="G"/>
+<pinref part="Q1" gate="G$1" pin="GATE"/>
 <pinref part="R36" gate="G$1" pin="2"/>
 <wire x1="43.18" y1="68.58" x2="45.72" y2="66.04" width="0.1524" layer="91"/>
